File: pcb/board_pf_cese/board_pf_cese.kicad_pcb (KiCad board)
At the start: 2 copper layers, 50 x 70 mm, 20 parts, among them J1 Screw_Terminal_01x02, J10 Screw_Terminal_01x02, J11 Conn_01x05, J2 Conn_01x04, J3 Conn_01x04, J4 Conn_01x04, J5 Conn_01x04, J6 Conn_01x15, J7 Conn_01x15, J8 Conn_01x08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

Commit message: update pcb
Parts:
- removed REF1, REF2, REF3, REF4: MountingHole_2mm, MountingHole:MountingHole_2mm
- added REF**: MountingHole_2.2mm_M2_Pad, MountingHole:MountingHole_2.2mm_M2_Pad, F.Cu at (146.0, 128.0)
- added REF**: MountingHole_2.2mm_M2_Pad, MountingHole:MountingHole_2.2mm_M2_Pad, F.Cu at (104.0, 66.0)
- added REF**: MountingHole_2.2mm_M2_Pad, MountingHole:MountingHole_2.2mm_M2_Pad, F.Cu at (104.0, 128.0)
- added REF**: MountingHole_2.2mm_M2_Pad, MountingHole:MountingHole_2.2mm_M2_Pad, F.Cu at (146.0, 66.0)
Other:
- outline, holes or cut-outs redrawn
Changed lines of the file:
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@@
   (net 46 "unconnected-(J11-Pin_4-Pad4)")
   (net 47 "unconnected-(J11-Pin_5-Pad5)")
+  (footprint "MountingHole:MountingHole_2.2mm_M2_Pad" (layer "F.Cu")
+    (at 146 128)
+    (descr "Mounting Hole 2.2mm, M2")
+    (tags "mounting hole 2.2mm m2")
+    (attr exclude_from_pos_files exclude_from_bom)
+    (fp_text reference "REF**" (at 0 -3.2) (layer "F.SilkS") hide
+        (effects (font (size 1 1) (thickness 0.15)))
+    )
+    (fp_text value "MountingHole_2.2mm_M2_Pad" (at 0 3.2) (layer "F.Fab")
+        (effects (font (size 1 1) (thickness 0.15)))
+    )
+    (fp_text user "${REFERENCE}" (at 0 0) (layer "F.Fab")
+        (effects (font (size 1 1) (thickness 0.15)))
+    )
+    (fp_circle (center 0 0) (end 2.2 0)
+      (stroke (width 0.15) (type solid)) (fill none) (layer "Cmts.User"))
+    (fp_circle (center 0 0) (end 2.45 0)
+      (stroke (width 0.05) (type solid)) (fill none) (layer "F.CrtYd"))
+    (pad "1" thru_hole circle (at 0 0) (size 4.4 4.4) (drill 2.2) (layers "*.Cu" "*.Mask"))
+  )
   (footprint "Connector_PinSocket_2.54mm:PinSocket_1x04_P2.54mm_Vertical" (layer "F.Cu")
     (at 129 127 90)
@@
     )
   )
-  (footprint "MountingHole:MountingHole_2mm" (layer "F.Cu")
-    (at 105 127)
-    (descr "Mounting Hole 2mm, no annular")
-    (tags "mounting hole 2mm no annular")
+  (footprint "MountingHole:MountingHole_2.2mm_M2_Pad" (layer "F.Cu")
+    (at 104 66)
+    (descr "Mounting Hole 2.2mm, M2")
+    (tags "mounting hole 2.2mm m2")
     (attr exclude_from_pos_files exclude_from_bom)
-    (fp_text reference "REF3" (at 0 -3) (layer "F.SilkS") hide
+    (fp_text reference "REF**" (at 0 -3.2) (layer "F.SilkS") hide
         (effects (font (size 1 1) (thickness 0.15)))
     )
-    (fp_text value "MountingHole_2mm" (at 0 3.1) (layer "F.Fab")
+    (fp_text value "MountingHole_2.2mm_M2_Pad" (at 0 3.2) (layer "F.Fab")
         (effects (font (size 1 1) (thickness 0.15)))
     )
@@
         (effects (font (size 1 1) (thickness 0.15)))
     )
-    (fp_circle (center 0 0) (end 2 0)
+    (fp_circle (center 0 0) (end 2.2 0)
       (stroke (width 0.15) (type solid)) (fill none) (layer "Cmts.User"))
-    (fp_circle (center 0 0) (end 2.25 0)
+    (fp_circle (center 0 0) (end 2.45 0)
       (stroke (width 0.05) (type solid)) (fill none) (layer "F.CrtYd"))
-    (pad "" np_thru_hole circle (at 0 0) (size 2 2) (drill 2) (layers "*.Cu" "*.Mask"))
+    (pad "1" thru_hole circle (at 0 0) (size 4.4 4.4) (drill 2.2) (layers "*.Cu" "*.Mask"))
   )
   (footprint "Resistor_THT:R_Axial_DIN0207_L6.3mm_D2.5mm_P10.16mm_Horizontal" (layer "F.Cu")
@@
     )
   )
-  (footprint "MountingHole:MountingHole_2mm" (layer "F.Cu")
-    (at 105 67)
-    (descr "Mounting Hole 2mm, no annular")
-    (tags "mounting hole 2mm no annular")
-    (attr exclude_from_pos_files exclude_from_bom)
-    (fp_text reference "REF1" (at 0 3.5) (layer "F.SilkS") hide
-        (effects (font (size 1 1) (thickness 0.15)))
-    )
-    (fp_text value "MountingHole_2mm" (at 0 3.1) (layer "F.Fab")
-        (effects (font (size 1 1) (thickness 0.15)))
-    )
-    (fp_text user "${REFERENCE}" (at 0 0) (layer "F.Fab")
-        (effects (font (size 1 1) (thickness 0.15)))
-    )
-    (fp_circle (center 0 0) (end 2 0)
-      (stroke (width 0.15) (type solid)) (fill none) (layer "Cmts.User"))
-    (fp_circle (center 0 0) (end 2.25 0)
-      (stroke (width 0.05) (type solid)) (fill none) (layer "F.CrtYd"))
-    (pad "" np_thru_hole circle (at 0 0) (size 2 2) (drill 2) (layers "*.Cu" "*.Mask"))
-  )
   (footprint "LED_THT:LED_D3.0mm" (layer "F.Cu")
     (at 139 86.46 -90)
@@
     )
   )
-  (footprint "MountingHole:MountingHole_2mm" (layer "F.Cu")
-    (at 145 127)
-    (descr "Mounting Hole 2mm, no annular")
-    (tags "mounting hole 2mm no annular")
+  (footprint "MountingHole:MountingHole_2.2mm_M2_Pad" (layer "F.Cu")
+    (at 104 128)
+    (descr "Mounting Hole 2.2mm, M2")
+    (tags "mounting hole 2.2mm m2")
     (attr exclude_from_pos_files exclude_from_bom)
-    (fp_text reference "REF4" (at 0 -3) (layer "F.SilkS") hide
+    (fp_text reference "REF**" (at 0 -3.2) (layer "F.SilkS") hide
         (effects (font (size 1 1) (thickness 0.15)))
     )
-    (fp_text value "MountingHole_2mm" (at 0 3.1) (layer "F.Fab")
+    (fp_text value "MountingHole_2.2mm_M2_Pad" (at 0 3.2) (layer "F.Fab")
         (effects (font (size 1 1) (thickness 0.15)))
     )
@@
         (effects (font (size 1 1) (thickness 0.15)))
     )
-    (fp_circle (center 0 0) (end 2 0)
+    (fp_circle (center 0 0) (end 2.2 0)
       (stroke (width 0.15) (type solid)) (fill none) (layer "Cmts.User"))
-    (fp_circle (center 0 0) (end 2.25 0)
+    (fp_circle (center 0 0) (end 2.45 0)
       (stroke (width 0.05) (type solid)) (fill none) (layer "F.CrtYd"))
-    (pad "" np_thru_hole circle (at 0 0) (size 2 2) (drill 2) (layers "*.Cu" "*.Mask"))
+    (pad "1" thru_hole circle (at 0 0) (size 4.4 4.4) (drill 2.2) (layers "*.Cu" "*.Mask"))
+  )
+  (footprint "MountingHole:MountingHole_2.2mm_M2_Pad" (layer "F.Cu")
+    (at 146 66)
+    (descr "Mounting Hole 2.2mm, M2")
+    (tags "mounting hole 2.2mm m2")
+    (attr exclude_from_pos_files exclude_from_bom)
+    (fp_text reference "REF**" (at 0 -3.2) (layer "F.SilkS") hide
+        (effects (font (size 1 1) (thickness 0.15)))
+    )
+    (fp_text value "MountingHole_2.2mm_M2_Pad" (at 0 3.2) (layer "F.Fab")
+        (effects (font (size 1 1) (thickness 0.15)))
+    )
+    (fp_text user "${REFERENCE}" (at 0 0) (layer "F.Fab")
+        (effects (font (size 1 1) (thickness 0.15)))
+    )
+    (fp_circle (center 0 0) (end 2.2 0)
+      (stroke (width 0.15) (type solid)) (fill none) (layer "Cmts.User"))
+    (fp_circle (center 0 0) (end 2.45 0)
+      (stroke (width 0.05) (type solid)) (fill none) (layer "F.CrtYd"))
+    (pad "1" thru_hole circle (at 0 0) (size 4.4 4.4) (drill 2.2) (layers "*.Cu" "*.Mask"))
   )
   (footprint "Connector_PinSocket_2.54mm:PinSocket_1x04_P2.54mm_Vertical" (layer "F.Cu")
@@
         (effects (font (size 1 1) (thickness 0.15)))
     )
-    (fp_text value "Conn_01x04" (at 2 28 90) (layer "F.Fab")
+    (fp_text value "Conn_01x04" (at 8 49 90) (layer "F.Fab") hide
         (effects (font (size 1 1) (thickness 0.15)))
     )
@@
     )
   )
-  (footprint "MountingHole:MountingHole_2mm" (layer "F.Cu")
-    (at 145 67)
-    (descr "Mounting Hole 2mm, no annular")
-    (tags "mounting hole 2mm no annular")
-    (attr exclude_from_pos_files exclude_from_bom)
-    (fp_text reference "REF2" (at -3.5 2.5) (layer "F.SilkS") hide
-        (effects (font (size 1 1) (thickness 0.15)))
-    )
-    (fp_text value "MountingHole_2mm" (at 0 3.1) (layer "F.Fab")
-        (effects (font (size 1 1) (thickness 0.15)))
-    )
-    (fp_text user "${REFERENCE}" (at 0 0) (layer "F.Fab")
-        (effects (font (size 1 1) (thickness 0.15)))
-    )
-    (fp_circle (center 0 0) (end 2 0)
-      (stroke (width 0.15) (type solid)) (fill none) (layer "Cmts.User"))
-    (fp_circle (center 0 0) (end 2.25 0)
-      (stroke (width 0.05) (type solid)) (fill none) (layer "F.CrtYd"))
-    (pad "" np_thru_hole circle (at 0 0) (size 2 2) (drill 2) (layers "*.Cu" "*.Mask"))
-  )
   (footprint "Connector_PinSocket_2.54mm:PinSocket_1x15_P2.54mm_Vertical" locked (layer "F.Cu")
     (at 142.56 116 -90)
@@
       (stroke (width 0.01) (type solid)) (fill solid) (layer "B.SilkS"))
   )
-  (gr_rect (start 100 62) (end 150 132)
-    (stroke (width 0.1) (type solid)) (fill none) (layer "Edge.Cuts"))
-  (gr_rect (start 102 64) (end 148 130)
-    (stroke (width 0.15) (type solid)) (fill none) (layer "Margin"))
+  (gr_arc (start 150 130) (mid 149.414214 131.414214) (end 148 132)
+    (stroke (width 0.1) (type default)) (layer "Edge.Cuts"))
+  (gr_arc (start 102 132) (mid 100.585786 131.414214) (end 100 130)
+    (stroke (width 0.1) (type default)) (layer "Edge.Cuts"))
+  (gr_arc (start 100 64) (mid 100.585786 62.585786) (end 102 62)
+    (stroke (width 0.1) (type default)) (layer "Edge.Cuts"))
+  (gr_line (start 102 62) (end 148 62)
+    (stroke (width 0.1) (type default)) (layer "Edge.Cuts"))
+  (gr_line (start 150 64) (end 150 130)
+    (stroke (width 0.1) (type default)) (layer "Edge.Cuts"))
+  (gr_arc (start 148 62) (mid 149.414214 62.585786) (end 150 64)
+    (stroke (width 0.1) (type default)) (layer "Edge.Cuts"))
+  (gr_line (start 100 130) (end 100 64)
+    (stroke (width 0.1) (type default)) (layer "Edge.Cuts"))
+  (gr_line (start 148 132) (end 102 132)
+    (stroke (width 0.1) (type default)) (layer "Edge.Cuts"))
+  (gr_rect (start 101 63) (end 149 131)
+    (stroke (width 0.15) (type default)) (fill none) (layer "Margin"))
   (gr_text "Ing. Mario Aguilar" (at 130.5 111.5) (layer "B.SilkS")
     (effects (font (size 1 1) (thickness 0.2) bold italic) (justify left bottom mirror))
