File: pcb/board_pf_cese/board_pf_cese.kicad_pcb (KiCad board)
At the start: 2 copper layers, 50 x 70 mm, 20 parts, among them J1 Screw_Terminal_01x02, J10 Screw_Terminal_01x02, J11 Conn_01x05, J2 Conn_01x04, J3 Conn_01x04, J4 Conn_01x04, J5 Conn_01x04, J6 Conn_01x15, J7 Conn_01x15, J8 Conn_01x08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

Commit message: finalizacion v1
Parts:
- removed the REF** at (124.0, 107.0)
- D1, D2: footprint LED_THT:LED_D3.0mm -> LED_THT:LED_D5.0mm
- J1, J10: footprint TerminalBlock_Phoenix:TerminalBlock_Phoenix_MPT-0,5-2-2.54_1x02_P2.54mm_Horizontal -> TerminalBlock_Phoenix:TerminalBlock_Phoenix_MKDS-1,5-2_1x02_P5.00mm_Horizontal
- moved R1 12.8 mm to (122.4, 97.0)
- moved D2 7.36 mm to (138.0, 93.8)
- moved D1 7.30 mm to (145.4, 93.8)
- moved J10 6.38 mm to (143.5, 87.9)
- moved J1 2.22 mm to (143.5, 76.7)
- moved R2 1.80 mm to (122.4, 93.0)
Routing:
- net /SCL: track 42.9 -> 22.9 mm
- net /UART2_TX: track 68.3 -> 50.0 mm, vias 1 -> 0
- net GND: track 12.2 -> 2.55 mm, vias 3 -> 0
- net Net-(D1-A): track 5.00 -> 14.1 mm
- net /M_TX: track 34.8 -> 40.3 mm
- net Net-(D2-A): track 11.2 -> 6.78 mm
- net /SDA: track 67.8 -> 63.9 mm
- net +5V: track 21.8 -> 18.4 mm
- net /SE: track 13.6 -> 15.9 mm
- net +12V: track 37.5 -> 36.5 mm
Other:
- board text added: "12V"
- board text added: "5V"
- board text added: "QUICK IoT BT_CESE"
- board text added: "UART_DEBUG"
- board text removed: "Ing. Mario Aguilar"

Commit message: actualizacion esquematico
Changed lines of the file:
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@@
       (layer "F.SilkS" (type "Top Silk Screen"))
       (layer "F.Paste" (type "Top Solder Paste"))
-      (layer "F.Mask" (type "Top Solder Mask") (color "Black") (thickness 0.01))
+      (layer "F.Mask" (type "Top Solder Mask") (color "Blue") (thickness 0.01))
       (layer "F.Cu" (type "copper") (thickness 0.035))
       (layer "dielectric 1" (type "core") (thickness 1.51) (material "FR4") (epsilon_r 4.5) (loss_tangent 0.02))
       (layer "B.Cu" (type "copper") (thickness 0.035))
-      (layer "B.Mask" (type "Bottom Solder Mask") (color "Black") (thickness 0.01))
+      (layer "B.Mask" (type "Bottom Solder Mask") (color "Blue") (thickness 0.01))
       (layer "B.Paste" (type "Bottom Solder Paste"))
       (layer "B.SilkS" (type "Bottom Silk Screen"))
@@
     (property "ki_keywords" "screw terminal")
     (attr through_hole)
-    (fp_text reference "J10" (at 2.5 -6.26 90) (layer "F.SilkS")
+    (fp_text reference "J10" (at 1.9 -6.5 90) (layer "F.SilkS")
         (effects (font (size 1 1) (thickness 0.15)))
     )
@@
     (effects (font (size 1.5 1.5) (thickness 0.3) bold) (justify bottom mirror))
   )
-  (gr_text "12V" (at 149.75 87 90) (layer "F.SilkS")
-    (effects (font (size 1 1) (thickness 0.15)) (justify left bottom))
-  )
-  (gr_text "5V" (at 150 75.25 90) (layer "F.SilkS")
-    (effects (font (size 1 1) (thickness 0.15)) (justify left bottom))
+  (gr_text "12V" (at 137.5 90.5 90) (layer "F.SilkS")
+    (effects (font (size 1 1) (thickness 0.125)) (justify left bottom))
+  )
+  (gr_text "5V" (at 137.5 72.5 90) (layer "F.SilkS")
+    (effects (font (size 1 1) (thickness 0.125)) (justify left bottom))
   )
   (gr_text "UART_DEBUG" (at 105.75 92.5) (layer "F.SilkS")
