File: pcb/board_pf_cese/board_pf_cese.kicad_sch (KiCad schematic)
At the start: 15 parts, among them J1 Screw_Terminal_01x02, J10 Screw_Terminal_01x02, J11 Conn_01x05, J2 Conn_01x04, J3 Conn_01x04, J4 Conn_01x04, J5 Conn_01x04, J6 Conn_01x15, J7 Conn_01x15, J8 Conn_01x08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

Commit message: actualizacion esquematico
Parts:
- removed D1, D2: LED, LED_THT:LED_D5.0mm, symbol Device:LED
- removed J1, J10: Screw_Terminal_01x02, TerminalBlock_Phoenix:TerminalBlock_Phoenix_MKDS-1,5-2_1x02_P5.00mm_Horizontal, symbol Connector:Screw_Terminal_01x02
- removed J11: Conn_01x05, Connector_PinSocket_2.54mm:PinSocket_1x05_P2.54mm_Vertical, symbol Connector_Generic:Conn_01x05
- removed J2, J3, J4, J5: Conn_01x04, Connector_PinSocket_2.54mm:PinSocket_1x04_P2.54mm_Vertical, symbol Connector_Generic:Conn_01x04
- removed J6, J7: Conn_01x15, Connector_PinSocket_2.54mm:PinSocket_1x15_P2.54mm_Vertical, symbol Connector_Generic:Conn_01x15
- removed J8, J9: Conn_01x08, Connector_PinSocket_2.54mm:PinSocket_1x08_P2.54mm_Vertical, symbol Connector_Generic:Conn_01x08
- removed R1, R2: R, Resistor_THT:R_Axial_DIN0207_L6.3mm_D2.5mm_P10.16mm_Horizontal, symbol Device:R
Connections:
- no-connect marks 30 -> 0
Other:
- added sheet Conectores_modulos (Conectores_modulos.kicad_sch)
- added sheet Debug (Debug.kicad_sch)
- added sheet conectores_alimentacion  (conectores_alimentacion .kicad_sch)
- added sheet conectores_sensores (conectores_sensores.kicad_sch)
- note added: "1"
- note added: "2"
- note added: "3"
- note added: "4"
- note added: "BOARD IMAGE BACK"
- note added: "BOARD IMAGE FRONT"
- note added: "BOARD_CESE_v01"
- note added: "CONECTORES ALIMENTACION"
- note added: "CONECTORES MODULOS"
- note added: "DEBUG"
- note added: "INDEX"
- note added: "PAGE #"
- note added: "VERSION: 01"
- note removed: "CONECTOR BATERIA 12V"
- note removed: "CONECTOR BATERIA 3.7V"
- note removed: "CONECTOR DEL MODULO NUCLEO-L432KC"
- note removed: "LEDS DE DEBUG"
- note removed: "MODULO DE COMUNICACION QUECTEL BG96"
- note removed: "UART2 DEBUG"
- note removed: "sensor de humedad AHT-10"
- note removed: "sensor de humedad de suelo"
- note removed: "sensor de humedad de suelo 2"
- note removed: "sensor de luz UV"
